File: PCB/Controller.kicad_pcb (KiCad board)
At the start: 2 copper layers, 120 x 92 mm, 134 parts, among them J1 Screw_Terminal_01x08, J2 Screw_Terminal_01x08, J3 PH, K1 TE_PCH-1xxx2M, K2 TE_PCH-1xxx2M, Q1 BCX56, Q2 BCX56, Q3 BCX56, Q4 BCX56, U1 WeMos S3 Mini, U10 MCP3208, U2 L7805, U3 MIC5504-3.3YM5, U4 MIC5504-3.3YM5, U5 OPA2991, U6 MCP3021, U7 ISO1640BDR, U8 OPA2991, U9 TL431D

Commit message: PCB Rev C in work
Parts:
- removed the D6 at (82.3, 88.9)
- removed the D7 at (86.4, 88.9)
- removed the REF** at (49.8, 81.5)
- added D14: BAT54, Package_TO_SOT_SMD:SOT-23, B.Cu at (72.9, 78.5)
- added D15: BAT54, Package_TO_SOT_SMD:SOT-23, B.Cu at (82.8, 78.7)
- added D16: BAT54, Package_TO_SOT_SMD:SOT-23, B.Cu at (65.5, 78.5)
- added J4: Screw_Terminal_01x08, Connector_Phoenix_MSTB:PhoenixContact_MSTBVA_2,5_8-G-5,08_1x08_P5.08mm_Vertical, B.Cu at (48.3, 86.9)
- added R52: 3.01k, Resistor_SMD:R_1206_3216Metric_Pad1.30x1.75mm_HandSolder, B.Cu at (76.2, 79.0)
- added R53: 3.01k, Resistor_SMD:R_1206_3216Metric_Pad1.30x1.75mm_HandSolder, B.Cu at (86.1, 79.2)
- added R54: 10k, Resistor_SMD:R_1206_3216Metric_Pad1.30x1.75mm_HandSolder, B.Cu at (68.8, 79.0)
- C1, C2: footprint Capacitor_THT:CP_Radial_D8.0mm_P2.50mm -> Capacitor_THT:CP_Radial_D10.0mm_P5.00mm
- R37, R38: value 10k -> na
- R41, R42: value 3.24k -> 10k
- U8: value OPA2991 -> MC34072
- moved R38 32.3 mm to (74.7, 122.9), turned to 90 degrees
- moved R37 30.6 mm to (71.1, 122.9), turned to 90 degrees
- moved R25 25.5 mm to (59.4, 100.8), turned to 180 degrees
- moved R23 24.0 mm to (59.4, 109.2), turned to 180 degrees
- moved R24 22.1 mm to (59.4, 106.4), turned to 0 degrees
- moved C10 21.8 mm to (59.4, 103.6), turned to 0 degrees
- moved R41 9.91 mm to (79.0, 79.0)
- moved R42 9.71 mm to (88.9, 79.2)
- moved C2 3.66 mm to (48.8, 128.2), turned to -90 degrees
- moved C1 3.52 mm to (59.9, 128.2), turned to -90 degrees
- moved R32 2.59 mm to (88.9, 98.6), turned to 180 degrees
- moved R33 2.59 mm to (74.7, 98.6), turned to 180 degrees
- moved R31 2.59 mm to (81.8, 98.6), turned to 180 degrees
- moved R34 2.59 mm to (67.6, 98.6), turned to 180 degrees
- moved D1 1.98 mm to (53.6, 132.6), turned to -90 degrees
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Connections:
- net Net-(J1-Pin_4) renamed /Relay1-NO
- net Net-(J1-Pin_6) renamed /Relay2-NO
- net Net-(J2-Pin_1) renamed /ADin1
- net Net-(J2-Pin_2) renamed /ADin2
- D4 pad 1: Net-(D4-K) -> Dout1
- D5 pad 1: Net-(D5-K) -> /Dout2
- J1 pad 3: Net-(J1-Pin_3) -> /Relay1-Com
- J1 pad 5: Net-(J1-Pin_5) -> /Relay2-Com
- J1 pad 7: Net-(D4-K) -> Dout1
- J1 pad 8: Net-(D5-K) -> /Dout2
- K1 pad 2: Net-(J1-Pin_3) -> /Relay1-Com
- K2 pad 2: Net-(J1-Pin_5) -> /Relay2-Com
- Q3 pad 2: Net-(D4-K) -> Dout1
- Q4 pad 2: Net-(D5-K) -> /Dout2
- R37 pad 1: Out1 -> /Relay1-Com
- R37 pad 2: Net-(D4-K) -> VS
- R38 pad 1: Out2 -> /Relay2-Com
- R38 pad 2: Net-(D5-K) -> VS
- R41 pad 1: GND -> In3
- R41 pad 2: Out1 -> Net-(J4-Pin_7)
- R42 pad 1: GND -> In4
- R42 pad 2: Out2 -> Net-(J4-Pin_8)
- U1 pad 15: unconnected-(U1-D44-Pad15) -> In2
- U1 pad 16: unconnected-(U1-D43-Pad16) -> In1
- U1 pad 17: In2 -> unconnected-(U1-D1-Pad17)
- U10 pad 7: Out1 -> In3
- U10 pad 8: Out2 -> In4
Routing:
- net VS: track 18.4 -> 138.4 mm
- net In2: track 36.8 -> 153.7 mm, vias 0 -> 4
- net Dout1: track 0.00 -> 88.3 mm, vias 0 -> 2
- net In1: track 40.3 -> 115.9 mm, vias 0 -> 2
- net Net-(D4-K): track 63.0 -> 0.00 mm
- net Net-(D5-K): track 57.1 -> 0.00 mm
- net +3.3V: track 203.7 -> 255.7 mm, vias 11 -> 13
- net SupV: track 109.3 -> 59.0 mm, vias 4 -> 2
- net /Dout2: track 0.00 -> 49.9 mm
- net In3: track 0.00 -> 32.8 mm, vias 0 -> 2
- net /Relay2-Com: track 0.00 -> 24.9 mm
- net /Relay1-Com: track 0.00 -> 24.1 mm
- net In4: track 0.00 -> 23.4 mm, vias 0 -> 2
- net Out1: track 22.6 -> 0.00 mm
- net Net-(J1-Pin_5): track 20.5 -> 0.00 mm
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
Commit message: SymbCtrl 2.9 work
Parts:
- added D17: BAT54, Package_TO_SOT_SMD:SOT-23, B.Cu at (153.7, 71.4)
- added D18: BAT54, Package_TO_SOT_SMD:SOT-23, B.Cu at (153.7, 67.6)
- added D19: BAT54, Package_TO_SOT_SMD:SOT-23, B.Cu at (118.6, 60.5)
- added J5: I2C Aux, Connector_Molex:Molex_KK-254_AE-6410-04A_1x04_P2.54mm_Vertical, F.Cu at (157.0, 73.2)
- added J6: One Wire, Connector_Molex:Molex_KK-254_AE-6410-03A_1x03_P2.54mm_Vertical, F.Cu at (115.3, 61.2)
- added R55: 10k, Resistor_SMD:R_1206_3216Metric_Pad1.30x1.75mm_HandSolder, B.Cu at (121.9, 60.2)
- C1, C2: value 47uF -> 330uF
- R31, R32, R33, R34: value 1k -> 270
- R37, R38: value na -> 0
- moved TP0 14.5 mm to (157.5, 83.8)
- moved REF** 4.83 mm to (68.3, 64.0)
- moved C6 3.70 mm to (153.9, 76.2)
- moved C3 1.54 mm to (154.3, 78.7)
Connections:
- U1 pad 17: unconnected-(U1-D1-Pad17) -> One
- U1 pad 8: unconnected-(U1-3V3-Pad8) -> +3.3VA
Routing:
- net +3.3VA: track 0.00 -> 86.5 mm, vias 0 -> 1
- net GND: track 161.2 -> 193.6 mm, vias 29 -> 30
- net One: track 0.00 -> 21.7 mm
- net SCL: track 49.2 -> 63.0 mm
- net SDA: track 45.5 -> 58.8 mm
- net DispD2: track 65.6 -> 62.8 mm
- net DispD1: track 65.4 -> 62.6 mm
- net DispD3: track 59.7 -> 57.1 mm
- net DispD0: track 71.3 -> 68.7 mm
- net DispE: track 71.1 -> 68.7 mm
- net DispD4: track 59.9 -> 57.5 mm
- net DispD5: track 54.0 -> 51.8 mm
- net DispRW: track 77.0 -> 74.9 mm
- net DispRS: track 76.8 -> 74.9 mm
- net DispD6: track 54.2 -> 52.2 mm
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
Commit message: Update to MBMon
Parts:
- U9: value TL431D -> TL431DBZ; footprint Package_SO:SOIC-8_3.9x4.9mm_P1.27mm -> Package_TO_SOT_SMD:SOT-23
- moved U9 1.61 mm to (108.0, 96.8), turned to 180 degrees
- moved R26 0.51 mm to (110.2, 93.2)
Connections:
- U9 pad 2: GND -> Net-(U10-Vref)
Routing:
- net GND: track 193.6 -> 188.5 mm, vias 30 -> 29
- net Net-(U10-Vref): track 16.0 -> 11.3 mm
- net +3.3V: track 255.7 -> 251.6 mm
