File: PCB/Controller.kicad_sch (KiCad schematic)
At the start: 126 parts, among them J1 Screw_Terminal_01x08, J2 Screw_Terminal_01x08, J3 PH, K1 TE_PCH-1xxx2M, K2 TE_PCH-1xxx2M, Q1 BCX56, Q2 BCX56, Q3 BCX56, Q4 BCX56, U1 WeMos S3 Mini, U10 MCP3208, U2 L7805, U3 MIC5504-3.3YM5, U4 MIC5504-3.3YM5, U5 OPA2991, U6 MCP3021, U7 ISO1640BDR, U8 MC34072, U9 TL431D

Commit message: PCB Rev C in work
Parts:
- added D14, D15, D16: BAT54, Package_TO_SOT_SMD:SOT-23, symbol Parts:BAT54SL
- added J4: Screw_Terminal_01x08, Connector_Phoenix_MSTB:PhoenixContact_MSTBVA_2,5_8-G-5,08_1x08_P5.08mm_Vertical, symbol Connector:Screw_Terminal_01x08
- added R37, R38: 0, Resistor_SMD:R_1206_3216Metric_Pad1.30x1.75mm_HandSolder, symbol Device:R_US
- added R41, R42, R54: 10k, Resistor_SMD:R_1206_3216Metric_Pad1.30x1.75mm_HandSolder, symbol Device:R_US
- added R52, R53: 3.01k, Resistor_SMD:R_1206_3216Metric_Pad1.30x1.75mm_HandSolder, symbol Device:R_US
- C1, C2: value 47uF -> 330uF; footprint Capacitor_THT:CP_Radial_D8.0mm_P2.50mm -> Capacitor_THT:CP_Radial_D10.0mm_P5.00mm
- R31, R32, R33, R34: value 1k -> 270
Connections:
- net +3.3V: now also D14.2 (K), D15.2 (K), D16.2 (K)
- net GND: now also D14.1 (A), D15.1 (A), D16.1 (A), J4.2 (Pin_2), R52.1, R53.1
- net In1: now also U1.16 (D43)
- net In2: now also U1.15 (D44), D16.3 (COM), D16.3 (COM), R54.1; no longer U1.17 (D1)
- net VS: now also J4.1 (Pin_1), J4.3 (Pin_3), J4.5 (Pin_5), R37.2, R38.2
- net ADin1: now reaches J2.1 (Pin_1), JP1.1 (A), R35.2
- net ADin2: now reaches J2.2 (Pin_2), JP2.1 (A), R36.2
- net Relay1-Com: now reaches J1.3 (Pin_3), K1.2
- net Relay1-Com: now also R37.1
- net Relay1-NO: now reaches J1.4 (Pin_4), K1.3
- net Relay2-Com: now reaches J1.5 (Pin_5), K2.2
- net Relay2-Com: now also R38.1
- net Relay2-NO: now reaches J1.6 (Pin_6), K2.3
- net Dout1: now reaches D4.1 (K), J1.7 (Pin_7), Q3.2 (C)
- net Dout1: now also J4.4 (Pin_4)
- net Dout2: now reaches D5.1 (K), J1.8 (Pin_8), Q4.2 (C)
- net Out1 renamed In3
- net In3: now also D14.3 (COM), D14.3 (COM), R41.1, R52.2
- net Out2 renamed In4
- net In4: now also D15.3 (COM), D15.3 (COM), R42.1, R53.2
- new net: J4.6 (Pin_6), R54.2
- new net: J4.8 (Pin_8), R42.2
- new net: J4.7 (Pin_7), R41.2
Other:
- note added: "2.7Vdc 10mA->"
- note added: "Ain/Din 1"
- note added: "Ain/Din 2"
- note added: "Ain/Din 3"
- note added: "Ain/Din 4"
- note added: "Dout 1"
- note added: "Dout 2"
- note added: "Gnd"
- note added: "Relay 1"
- note added: "Relay 2"
- note added: "T1in"
- note added: "T1ref"
- note added: "T2in"
- note added: "T2ref"
- note added: "VSupply"
- note added: "Vsupply"
- note removed: "2.1Vdc 1.2mA-->"
- moved on the sheet: C24, C25, C26, C27, C28, D10A, D10B, D11A, D11B, D12A, D12B, D13A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

Commit message: SymbCtrl 2.9 work
Parts:
- added D17, D18, D19: BAT54, Package_TO_SOT_SMD:SOT-23, symbol Parts:BAT54SL
- added J5: I2C Aux, Connector_Molex:Molex_KK-254_AE-6410-04A_1x04_P2.54mm_Vertical, symbol Connector_Generic:Conn_01x04
- added J6: One Wire, Connector_Molex:Molex_KK-254_AE-6410-03A_1x03_P2.54mm_Vertical, symbol Connector_Generic:Conn_01x03
- added R55: 10k, Resistor_SMD:R_1206_3216Metric_Pad1.30x1.75mm_HandSolder, symbol Device:R_US
Connections:
- net GND: now also D17.1 (A), D18.1 (A), D19.1 (A), J5.4 (Pin_4), J6.3 (Pin_3)
- net SCL: now also D18.3 (COM), D18.3 (COM), J5.3 (Pin_3)
- net SDA: now also D17.3 (COM), D17.3 (COM), J5.2 (Pin_2)
- net One: now reaches U1.17 (D1)
- net One: now also D19.3 (COM), D19.3 (COM), J6.2 (Pin_2), R55.1
- net +3.3VA: now reaches U1.8 (3V3)
- net +3.3VA: now also D17.2 (K), D18.2 (K), D19.2 (K), J5.1 (Pin_1), J6.1 (Pin_1), R55.2
Other:
- note added: "10mA->"
- note removed: "2.7Vdc 10mA->"
- moved on the sheet: DS1, R51

Commit message: Update to MBMon
Parts:
- removed U9: TL431D, Package_SO:SOIC-8_3.9x4.9mm_P1.27mm, symbol Reference_Voltage:TL431D
- added U9: TL431DBZ, Package_TO_SOT_SMD:SOT-23, symbol Reference_Voltage:TL431DBZ
Connections:
- net GND: now also U9.3 (A)
- net at R26.2, U10.15 (Vref): now also U9.1 (K), U9.2 (REF)
Changed lines of the file:
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@@
+    )
+  )
+  (symbol (lib_id "Reference_Voltage:TL431DBZ") (at 274.32 189.23 270) (mirror x) (unit 1)
+    (in_bom yes) (on_board yes) (dnp no) (fields_autoplaced)
+    (property "Reference" "U9" (at 271.78 187.96 90)
+      (effects (font (size 1.27 1.27)) (justify right))
+    )
+    (property "Value" "TL431DBZ" (at 271.78 190.5 90)
+      (effects (font (size 1.27 1.27)) (justify right))
+    )
+    (property "Footprint" "Package_TO_SOT_SMD:SOT-23" (at 270.51 189.23 0)
+      (effects (font (size 1.27 1.27) italic) hide)
+    )
+    (property "Datasheet" "http://www.ti.com/lit/ds/symlink/tl431.pdf" (at 274.32 189.23 0)
+      (effects (font (size 1.27 1.27) italic) hide)
+    )
+    (pin "1")
+    (pin "2")
+    (pin "3")
+    (instances
+      (project "Controller"
+        (path "/e98a57d9-3732-4e84-8c7e-17ff22fc8918"
+          (reference "U9") (unit 1)
+        )
+      )
     )
   )
@@
         )
       )
-    )
-  )
-  (symbol (lib_id "Reference_Voltage:TL431D") (at 274.32 189.23 270) (mirror x) (unit 1)
-    (in_bom yes) (on_board yes) (dnp no) (fields_autoplaced)
-    (property "Reference" "U9" (at 271.78 187.96 90)
-      (effects (font (size 1.27 1.27)) (justify right))
-    )
-    (property "Value" "TL431D" (at 271.78 190.5 90)
-      (effects (font (size 1.27 1.27)) (justify right))
-    )
-    (property "Footprint" "Package_SO:SOIC-8_3.9x4.9mm_P1.27mm" (at 267.97 189.23 0)
-      (effects (font (size 1.27 1.27) italic) hide)
-    )
-    (property "Datasheet" "http://www.ti.com/lit/ds/symlink/tl431.pdf" (at 274.32 189.23 0)
-      (effects (font (size 1.27 1.27) italic) hide)
-    )
-    (pin "1")
-    (pin "2")
-    (pin "3")
-    (pin "6")
-    (pin "7")
-    (pin "8")
-    (instances
-      (project "Controller"
-        (path "/e98a57d9-3732-4e84-8c7e-17ff22fc8918"
-          (reference "U9") (unit 1)
-        )
-      )
